Commit message: Base working
Momentum slider that can apply force, creating constraint works

File: pendulum_climb/assets/pendulum.urdf (robot description, URDF)
Before this commit: robot pendulum, 3 links, 2 joints
Joints:
- joint bottom_joint: axis 0 0 0 -> 1 0 0; limit (none) -> effort=1000 velocity=100; type fixed -> continuous
- joint top_joint: axis 0 0 0 -> 1 0 0; limit (none) -> effort=1000 velocity=100; type fixed -> continuous

File: pendulum_climb/assets/target.urdf (robot description, URDF)
Before this commit: robot target, 1 links, 0 joints
Links:
- link base_link: geometry visual sphere length=1 radius=0.05

Commit message: initial revision

File: pendulum_climb/assets/pendulum.urdf (robot description, URDF)
Before this commit: robot pendulum, 3 links, 2 joints
Links:
- link base_link: geometry collision capsule length=1.5 radius=0.2; visual capsule length=1.5 radius=0.2
Joints:
- joint bottom_joint: axis 1 0 0 -> 0 0 0; limit effort=1000 velocity=100 -> lower=0 upper=0 effort=0.0 velocity=0.0; origin xyz=0 0 -0.5 -> xyz=0 0 -1.0; type continuous -> fixed
- joint top_joint: axis 1 0 0 -> 0 0 0; limit effort=1000 velocity=100 -> lower=0 upper=0 effort=0.0 velocity=0.0; origin xyz=0 0 0.5 -> xyz=0 0 1.0; type continuous -> spherical

Commit message: info and action adjustments
actions reverted back to moving only +/- x

File: pendulum_climb/assets/pendulum.urdf (robot description, URDF)
Before this commit: robot pendulum, 3 links, 2 joints
Joints:
- joint top_joint: type spherical -> fixed
